File: hardware/kicad/habit-calendar.kicad_sch (KiCad schematic)
At the start: 0 parts

Commit message: Sent to production!
Other:
- sheet habit-calender-subsheet-for-replica ports: added inLed, outLed; removed none
- sheet habit-calender-subsheet-for-replica1 ports: added inLed, outLed; removed none
Changed lines of the file:
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@@
+    (stroke (width 0) (type default) (color 0 0 0 0))
+  )
+  (wire (pts (xy 149.86 84.2772) (xy 150.495 84.2772))
     (stroke (width 0) (type default) (color 0 0 0 0))
   )
@@
       (effects (font (size 1.27 1.27)) (justify left))
     )
+    (pin "outLed" output (at 149.86 84.2772 0)
+      (effects (font (size 1.27 1.27)) (justify right))
+    )
+    (pin "inLed" input (at 123.3424 84.0994 180)
+      (effects (font (size 1.27 1.27)) (justify left))
+    )
   )
   (sheet (at 150.495 72.771) (size 26.5176 12.3444) (fields_autoplaced)
@@
       (effects (font (size 1.27 1.27)) (justify left))
     )
+    (pin "outLed" output (at 177.0126 84.328 0)
+      (effects (font (size 1.27 1.27)) (justify right))
+    )
+    (pin "inLed" input (at 150.495 84.2772 180)
+      (effects (font (size 1.27 1.27)) (justify left))
+    )
